File: plate/plate.kicad_pcb (KiCad board)
At the start: 2 copper layers, 338.1 x 143.8 mm, 0 parts

Commit message: Actually trace the correct line for the plate
Other:
- board size 338.1 x 143.8 mm -> 348.1 x 153.8 mm
