File: plate/plate.kicad_pcb (KiCad board)
At the start: 2 copper layers, 348.1 x 153.8 mm, 0 parts

Commit message: Reduce gap between plate feet and plate to 2mm
Other:
- board size 348.1 x 153.8 mm -> 348.1 x 147.8 mm

Commit message: Shorten plate correspondingly
Other:
- board size 348.1 x 147.8 mm -> 348.1 x 137.8 mm
